File: TMS9918A Video Card.kicad_sch (KiCad schematic)
At the start: 15 parts

Commit message: Schematic cleanup
Parts:
- C1, C10, C13: value (none) -> 0.1µF; footprint (none) -> Capacitor_THT:C_Disc_D5.0mm_W2.5mm_P2.50mm
- C11, C12: value (none) -> 27pF; footprint (none) -> Capacitor_THT:C_Disc_D3.8mm_W2.6mm_P2.50mm
- FB1: value (none) -> FerriteBead_Small; footprint (none) -> Ferrite_THT:LairdTech_28C0236-0JW-10
- J1: value (none) -> Video Out; footprint (none) -> Connector_Audio:Jack_RCA_CUI_RCJ-04
- J2: value (none) -> Video Out; footprint (none) -> Connector_PinHeader_2.54mm:PinHeader_1x02_P2.54mm_Vertical
- J4: value (none) -> Edge Connector; footprint (none) -> Connector_PCBEdge:Interis_Expansion_PCBEdge
- Q1: value (none) -> 2N4401; footprint (none) -> Package_TO_SOT_THT:TO-92_Inline
- R1: value (none) -> 470; footprint (none) -> Resistor_THT:R_Axial_DIN0207_L6.3mm_D2.5mm_P10.16mm_Horizontal
- R2: value (none) -> 75; footprint (none) -> Resistor_THT:R_Axial_DIN0207_L6.3mm_D2.5mm_P10.16mm_Horizontal
- U1: value (none) -> TMS9918A; footprint (none) -> Package_DIP:DIP-40_W15.24mm
- U10: value (none) -> 74LS32; footprint (none) -> Package_DIP:DIP-14_W7.62mm
- X1: value (none) -> 10.738635 MHz; footprint (none) -> Crystal:Crystal_HC49-U_Vertical
Other:
- sheet dram renamed RAM
