File: dram.kicad_sch (KiCad schematic)
At the start: 16 parts, among them U2 4164, U3 4164, U4 4164, U5 4164, U6 4164, U7 4164, U8 4164, U9 4164

Commit message: Schematic cleanup
Parts:
- C2, C3, C4, C5, C6, C7, C8, C9: value (none) -> 0.1µF; footprint (none) -> Capacitor_THT:C_Disc_D5.0mm_W2.5mm_P2.50mm
- U2, U3, U4, U5, U6, U7, U8, U9: footprint (none) -> Package_DIP:DIP-16_W7.62mm
Other:
- moved on the sheet: C2, C3, C4, C5, C6, C7, C8, C9, U2, U3, U4, U5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
